Commit message: Fix camera position

File: sim_env_ws/src/arm_description/urdf/arm_stand.urdf (robot description, URDF)
Before this commit: robot arm_stand, 48 links, 47 joints
Links:
- link camera_link: geometry collision box size=0.05 0.05 0.05; visual box size=0.05 0.05 0.05
Joints:
- joint camera_joint: axis 1 0 0 -> (none); origin (none) -> xyz=0 0 0.4 rpy=0 1.57 -1.57; type continuous -> fixed
- joint hand_palm_joint: parent camera_link -> top_link
- joint hand_safety_box_joint: parent camera_link -> top_link
- joint hand_tool_joint: parent camera_link -> top_link

File: sim_env_ws/src/arm_description/urdf/arm_stand.urdf.xacro (robot description, xacro)
@@ -9,9 +9,10 @@
   <xacro:property name="axle_offset" value="0.05" />
   <xacro:property name="damp" value="0.7" />
-  <xacro:property name="camera_link" value="0.05" /> <!-- Size of square 'camera' box -->
+  <xacro:property name="camera_link" value="0.05" />
+  <!-- Size of square 'camera' box -->
   <!-- Import Rviz colors -->
   <xacro:include
       filename="$(find arm_description)/urdf/materials.urdf.xacro" />
-  <!--< Default Inertial
+  <!-- Default Inertial -->
   <xacro:macro name="default_inertial" params="z_value i_value mass">
     <inertial>
@@ -22,5 +23,5 @@
                izz="${i_value}" />
     </inertial>
-  </xacro:macro> -->
+  </xacro:macro>
   <!-- Importing End-Effector -->
   <!--Arguments-->
@@ -32,5 +33,5 @@
   <xacro:include filename="$(find tiago_description)/urdf/end_effector/end_effector.urdf.xacro" />
   <xacro:include filename="$(find tiago_description_calibration)/urdf/calibration/calibration_constants.urdf.xacro" />
-  <xacro:tiago_end_effector name="${end_effector_name}" parent="camera_link" type="${end_effector}" reflect="1"/>
+  <xacro:tiago_end_effector name="${end_effector_name}" parent="top_link" type="${end_effector}" reflect="1"/>
   <!-- Include Gazebo tags -->
   <xacro:include filename="$(find arm_description)/gazebo/arm_stand_gazebo.urdf.xacro"/>
@@ -56,14 +57,5 @@
       </geometry>
     </collision>
-    <inertial>
-      <origin xyz="0 0 ${height1/2}" rpy="0 0 0"/>
-      <mass value="1"/>
-      <inertia
-        ixx="1.0" ixy="0.0" ixz="0.0"
-        iyy="1.0" iyz="0.0"
-        izz="1.0"/>
-    </inertial>
-    <!-- <xacro:default_inertial z_value="${height1/2}"
-    i_value="1.0" mass="1"/> -->
+    <xacro:default_inertial z_value="${height1/2}" i_value="1.0" mass="1"/>
   </link>
   <!-- Joint between Base Link and Middle Link -->
@@ -91,14 +83,6 @@
       </geometry>
     </collision>
-    <inertial>
-      <origin xyz="0 0 ${height2/2 - axle_offset}" rpy="0 0 0"/>
-      <mass value="1"/>
-      <inertia
-        ixx="1.0" ixy="0.0" ixz="0.0"
-        iyy="1.0" iyz="0.0"
-        izz="1.0"/>
-    </inertial>
-    <!-- <xacro:default_inertial z_value="${height2/2 - axle_offset}"
-      i_value="1.0" mass="1"/> -->
+    <xacro:default_inertial z_value="${height2/2 - axle_offset}"
+    i_value="1.0" mass="1"/>
   </link>
   <!-- Joint between Middle Link and Top Link 3DOF -->
@@ -165,18 +149,9 @@
       </geometry>
     </collision>
-    <inertial>
-      <origin xyz="0 0 ${height3/2 - axle_offset}" rpy="0 0 0"/>
-      <mass value="1"/>
-      <inertia
-        ixx="1.0" ixy="0.0" ixz="0.0"
-        iyy="1.0" iyz="0.0"
-        izz="1.0"/>
-    </inertial>
-    <!--< xacro:default_inertial z_value="${height3/2 - axle_offset}"
-      i_value="1.0" mass="1"/> -->
+    <xacro:default_inertial z_value="${height3/2 - axle_offset}"
+      i_value="1.0" mass="1"/>
   </link>
   <joint name="camera_joint" type="fixed">
-    <axis xyz="1 0 0" />
-    <origin xyz="${camera_link} 0 ${height3 - axle_offset*2}" rpy="0 0 0"/>
+    <origin xyz="0 0 ${height2 - axle_offset*2}" rpy="0 1.57 -1.57"/>
     <parent link="top_link"/>
     <child link="camera_link"/>
@@ -187,11 +162,11 @@
       <origin xyz="0 0 0" rpy="0 0 0"/>
       <geometry>
-    <box size="${camera_link} ${camera_link} ${camera_link}"/>
+        <box size="${camera_link} ${camera_link} ${camera_link}"/>
       </geometry>
     </collision>
     <visual>
-      <origin xyz="0 0 0" rpy="0 0 0"/>
+      <origin xyz="0 0 ${camera_link + axle_offset/2}" rpy="0 0 0"/>
       <geometry>
-    <box size="${camera_link} ${camera_link} ${camera_link}"/>
+        <box size="${camera_link} ${camera_link} ${camera_link}"/>
       </geometry>
       <material name="white"/>
