Commit message: attach tiago hand to arm stand

File: sim_env_ws/src/arm_description/urdf/arm_stand.urdf.xacro (robot description, xacro)
@@ -4,7 +4,7 @@
   <!-- Constants for robot dimensions -->
   <xacro:property name="width" value="0.1" />
-  <xacro:property name="height1" value="2" />
-  <xacro:property name="height2" value="1" />
-  <xacro:property name="height3" value="1" />
+  <xacro:property name="height1" value="1" />
+  <xacro:property name="height2" value="0.5" />
+  <xacro:property name="height3" value="0.5" />
   <xacro:property name="axle_offset" value="0.05" />
   <xacro:property name="damp" value="0.7" />
@@ -22,5 +22,14 @@
     </inertial>
   </xacro:macro>
+  <!-- Importing End-Effector -->
+  <!--Arguments-->
+  <xacro:arg name="end_effector" default="pal-hey5"/> <!-- false, pal-gripper, pal-hey5, schunk-wsg-->
+  <xacro:property name="end_effector" value="$(arg end_effector)" />
+  <xacro:property name="end_effector_name"       value="${'hand' if end_effector == 'pal-hey5' else 'gripper'}"/>
+  <!-- Include end effector -->
   <!--<xacro:include filename="$(find hey5_description)/urdf/gripper.xacro"/>-->
+  <xacro:include filename="$(find tiago_description)/urdf/end_effector/end_effector.urdf.xacro" />
+  <xacro:include filename="$(find tiago_description_calibration)/urdf/calibration/calibration_constants.urdf.xacro" />
+  <xacro:tiago_end_effector name="${end_effector_name}" parent="top_link" type="${end_effector}" reflect="1"/>
   <link name="dummy">
    </link>
@@ -101,4 +110,11 @@
       i_value="1.0" mass="1"/>
   </link>
+ <!-- <joint name="hand_joint" type="revolute">
+    <parent link="top_link"/>
+    <child link="left_gripper"/>
+    <origin xyz="0 0 ${height2 - axle_offset}" rpy="0 -1.57 0"/>
+    <axis xyz="0 0 1"/>
+    <limit effort="30.0" lower="-0.548" upper="0.0" velocity="0.1"/>
+  </joint> -->
 </robot>
 <!--

File: sim_env_ws/src/tiago_description_complete/tiago_robot/tiago_description/urdf/end_effector/end_effector.urdf.xacro (robot description, xacro)
@@ -44,10 +44,12 @@
   <xacro:if value="${type == 'pal-hey5'}">
     <xacro:hey5_hand parent="${parent}" name="${name}" reflect="${reflect}">
-      <origin xyz="0 0 0" rpy="0 0 0"/>
+      <origin xyz="0 0 ${height2 - axle_offset}" rpy="0 -1.57 0"/>
+      <!--<origin xyz="0 0 0" rpy="0 0 0"/>-->
     </xacro:hey5_hand>
     <joint name="${name}_safety_box_joint" type="fixed">
       <parent link="${parent}"/>
       <child link="${name}_safety_box"/>
-      <origin xyz="0.1 0.02 ${reflect * 0.02}" rpy="0 0 0"/>
+      <origin xyz="0 0 ${height2 - axle_offset}" rpy="0 -1.57 0"/>
+      <!--<origin xyz="0.1 0.02 ${reflect * 0.02}" rpy="0 0 0"/>-->
     </joint>
     <link name="${name}_safety_box">

Commit message: made mid-top joint 3 DOF (ball & socket)

File: sim_env_ws/src/arm_description/urdf/arm_stand.urdf.xacro (robot description, xacro)
@@ -83,12 +83,33 @@
       i_value="1.0" mass="1"/>
   </link>
-  <!-- Joint between Middle Link and Top Link -->
-  <joint name="joint_mid_top" type="revolute">
+  <!-- Joint between Middle Link and Top Link 3DOF -->
+  <joint name="joint_mid_top" type="fixed">
     <parent link="mid_link" />
-    <child link="top_link" />
+    <child link="ball_link" />
     <origin xyz="0 ${width} ${height2 - axle_offset*2}" rpy="0 0 0"/>
-    <axis xyz="0 1 0" />
+    <!--<axis xyz="0 1 0" />
     <dynamics damping="${damp}" />
-    <limit effort="100.0" velocity="0.5" lower="-3.14" upper="3.14"/>
+    <limit effort="100.0" velocity="0.5" lower="-3.14" upper="3.14"/>-->
+  </joint>
+  <link name="ball_link" />
+  <joint name="joint_mid_top_psi" type="continuous" >
+      <parent link="ball_link" />
+      <child link="ball_link_psi_link" />
+      <axis xyz="0 0 1" />
+      <dynamics damping="${damp}" />
+  </joint>
+  <link name="ball_link_psi_link" />
+  <joint name="joint_mid_top_theta" type="continuous" >
+      <parent link="ball_link_psi_link"/>
+      <child link="ball_link_theta_link"/>
+      <axis xyz="0 1 0" />
+      <dynamics damping="${damp}" />
+  </joint>
+  <link name="ball_link_theta_link" />
+  <joint name="joint_mid_top__phi" type="continuous" >
+      <parent link="ball_link_theta_link"/>
+      <child link="top_link"/>
+      <axis xyz="1 0 0" />
+      <dynamics damping="${damp}" />
   </joint>
   <!-- Top Link -->

Commit message: Attach tiago hand to arm stand + insert into our startup_world in Gazebo

File: sim_env_ws/src/arm_description/urdf/arm_stand.urdf.xacro (robot description, xacro)
@@ -32,6 +32,12 @@
   <xacro:include filename="$(find tiago_description_calibration)/urdf/calibration/calibration_constants.urdf.xacro" />
   <xacro:tiago_end_effector name="${end_effector_name}" parent="top_link" type="${end_effector}" reflect="1"/>
-  <link name="dummy">
-   </link>
+  <!-- Include Gazebo tags -->
+  <xacro:include filename="$(find arm_description)/gazebo/arm_stand_gazebo.urdf.xacro"/>
+  <!--Arm Stand-->
+  <link name="world"/>
+  <joint name="fixed" type="fixed">
+    <parent link="world"/>
+    <child link="base_link"/>
+  </joint>
   <!-- Base Link -->
   <link name="base_link">
@@ -52,8 +58,4 @@
     i_value="1.0" mass="1"/>
   </link>
-  <joint name="dummy_joint" type="fixed">
-     <parent link="dummy"/>
-     <child link="base_link"/>
-   </joint>
   <!-- Joint between Base Link and Middle Link -->
   <joint name="joint_base_mid" type="revolute">
@@ -92,5 +94,11 @@
     <limit effort="100.0" velocity="0.5" lower="-3.14" upper="3.14"/>-->
   </joint>
-  <link name="ball_link" />
+  <link name="ball_link">
+    <inertial>
+      <origin xyz="0 0 0" rpy="0 0 0"/>
+      <mass value=".00001"/>
+      <inertia ixx="0.00001" ixy="0.0" ixz="0.0" iyy="0.00001"  iyz="0.0" izz ="0.00001"/>
+    </inertial>
+  </link>
   <joint name="joint_mid_top_psi" type="continuous" >
       <parent link="ball_link" />
@@ -99,5 +107,11 @@
       <dynamics damping="${damp}" />
   </joint>
-  <link name="ball_link_psi_link" />
+  <link name="ball_link_psi_link" >
+    <inertial>
+      <origin xyz="0 0 0" rpy="0 0 0"/>
+      <mass value=".00001"/>
+      <inertia ixx="0.00001" ixy="0.0" ixz="0.0" iyy="0.000011"  iyz="0.0" izz ="0.00001"/>
+    </inertial>
+  </link>
   <joint name="joint_mid_top_theta" type="continuous" >
       <parent link="ball_link_psi_link"/>
@@ -106,5 +120,11 @@
       <dynamics damping="${damp}" />
   </joint>
-  <link name="ball_link_theta_link" />
+  <link name="ball_link_theta_link" >
+    <inertial>
+      <origin xyz="0 0 0" rpy="0 0 0"/>
+      <mass value=".00001"/>
+      <inertia ixx="0.00001" ixy="0.0" ixz="0.0" iyy="0.00001"  iyz="0.0" izz ="0.00001"/>
+    </inertial>
+  </link>
   <joint name="joint_mid_top__phi" type="continuous" >
       <parent link="ball_link_theta_link"/>

Commit message: connection successful between gazebo and moveit BUT execution fails acc to moveit due to discrepancies between ros controllers in gazebo and moveit

File: sim_env_ws/src/arm_description/urdf/arm_stand.urdf.xacro (robot description, xacro)
@@ -41,5 +41,5 @@
   <!--Arm Stand-->
   <link name="world"/>
-  <joint name="fixed" type="fixed">
+  <joint name="virtual_joint" type="fixed">
     <parent link="world"/>
     <child link="base_link"/>

Commit message: adjusting some launch files

File: sim_env_ws/src/arm_description/urdf/arm_stand.urdf.xacro (robot description, xacro)
@@ -10,5 +10,5 @@
   <xacro:property name="height3" value="0.5" />
   <xacro:property name="axle_offset" value="0.05" />
-  <xacro:property name="damp" value="0.7" />
+  <xacro:property name="damp" value="0.1" /> <!--0.7 damp and vel limit 0.5-->
   <xacro:property name="friction" value="0" />
   <xacro:property name="camera_link" value="0.05" />
@@ -69,5 +69,5 @@
     <axis xyz="0 1 0" />
     <dynamics damping="${damp}" friction = "${friction}" />
-    <limit effort="1000.0" velocity="0.5" lower="-3.14" upper="3.14"/>
+    <limit effort="1000.0" velocity="1" lower="-3.14" upper="3.14"/>
   </joint>
   <!-- Middle Link -->
@@ -96,5 +96,5 @@
     <axis xyz="0 0 1" />
     <dynamics damping="${damp}" friction = "${friction}" />
-    <limit effort="1000.0" velocity="0.5" lower="-3.14" upper="3.14"/>
+    <limit effort="1000.0" velocity="1" lower="-3.14" upper="3.14"/>
   </joint>
   <!-- Top Link -->
@@ -128,5 +128,5 @@
     <axis xyz="1 0 0" />
     <dynamics damping="${damp}" friction = "${friction}" />
-    <limit effort="1000.0" velocity="0.5" lower="-3.14" upper="3.14"/>
+    <limit effort="1000.0" velocity="1" lower="-3.14" upper="3.14"/>
   </joint>
   <link name="fore_link">

Commit message: added demo scriptreadme file

File: sim_env_ws/src/arm_description/urdf/arm_stand.urdf.xacro (robot description, xacro)
@@ -6,4 +6,5 @@
   <xacro:property name="mass" value="1" />
   <xacro:property name="width" value="0.1" />
+  <xacro:property name="width3" value="0.15" />
   <xacro:property name="height1" value="1" />
   <xacro:property name="height2" value="0.5" />
@@ -134,5 +135,5 @@
       <origin xyz="${height3/2} 0 0" rpy="0 0 0" />
       <geometry>
-        <box size="${height3} ${width} ${width}" />
+        <box size="${height3} ${width} ${width3}" />
       </geometry>
       <material name="blue"/>
@@ -141,5 +142,5 @@
       <origin xyz="${height3/2} 0 0" rpy="0 0 0" />
       <geometry>
-        <box size="${height3} ${width} ${width}" />
+        <box size="${height3} ${width} ${width3}" />
       </geometry>
     </collision>
@@ -161,5 +162,5 @@
   <link name="camera_link">
     <collision>
-      <origin xyz="0 0 ${camera_link + camera_link/2}" rpy="0 0 0"/>
+      <origin xyz="0 0 ${camera_link + camera_link/2 + 0.05/2}" rpy="0 0 0"/>
       <geometry>
         <box size="${camera_link} ${camera_link} ${camera_link}"/>
@@ -167,5 +168,5 @@
     </collision>
     <visual>
-      <origin xyz="0 0 ${camera_link + camera_link/2}" rpy="0 0 0"/>
+      <origin xyz="0 0 ${camera_link + camera_link/2 +0.05/2}" rpy="0 0 0"/>
       <geometry>
         <box size="${camera_link} ${camera_link} ${camera_link}"/>
