Commit message: add camera link to the arm

File: sim_env_ws/src/arm_description/gazebo/arm_stand_gazebo.urdf.xacro (robot description, xacro)
@@ -24,3 +24,42 @@
     </plugin>
   </gazebo>-->
+  <gazebo reference="camera_link">
+    <sensor type="camera" name="camera1">
+      <update_rate>30.0</update_rate>
+      <camera name="camera1">
+        <horizontal_fov>1.3962634</horizontal_fov>
+        <image>
+          <width>800</width>
+          <height>800</height>
+          <format>R8G8B8</format>
+        </image>
+        <clip>
+          <near>0.02</near>
+          <far>300</far>
+        </clip>
+        <noise>
+          <type>gaussian</type>
+          <!-- Noise is sampled independently per pixel on each frame.
+               That pixel's noise value is added to each of its color
+               channels, which at that point lie in the range [0,1]. -->
+          <mean>0.0</mean>
+          <stddev>0.007</stddev>
+        </noise>
+      </camera>
+      <plugin name="camera_controller" filename="libgazebo_ros_camera.so">
+        <alwaysOn>true</alwaysOn>
+        <updateRate>0.0</updateRate>
+        <cameraName>camera1</cameraName>
+        <imageTopicName>image_raw</imageTopicName>
+        <cameraInfoTopicName>camera_info</cameraInfoTopicName>
+        <frameName>camera_link</frameName>
+        <hackBaseline>0.07</hackBaseline>
+        <distortionK1>0.0</distortionK1>
+        <distortionK2>0.0</distortionK2>
+        <distortionK3>0.0</distortionK3>
+        <distortionT1>0.0</distortionT1>
+        <distortionT2>0.0</distortionT2>
+      </plugin>
+    </sensor>
+  </gazebo>
 </robot>

File: sim_env_ws/src/arm_description/urdf/arm_stand.urdf (robot description, URDF)
Before this commit: robot arm_stand, 47 links, 46 joints
Links:
- added link camera_link, mass 1e-5; collision box size=${camera_link} ${camera_link} ${camera_link}; visual box size=${camera_link} ${camera_link} ${camera_link}
Joints:
- added joint camera_joint: type continuous, parent top_link, child camera_link, axis 1 0 0
- joint hand_palm_joint: parent top_link -> camera_link
- joint hand_safety_box_joint: parent top_link -> camera_link
- joint hand_tool_joint: parent top_link -> camera_link

File: sim_env_ws/src/arm_description/urdf/arm_stand.urdf.xacro (robot description, xacro)
@@ -9,8 +9,9 @@
   <xacro:property name="axle_offset" value="0.05" />
   <xacro:property name="damp" value="0.7" />
+  <xacro:property name="camera_link" value="0.05" /> <!-- Size of square 'camera' box -->
   <!-- Import Rviz colors -->
   <xacro:include
       filename="$(find arm_description)/urdf/materials.urdf.xacro" />
-  <!-- Default Inertial -->
+  <!--< Default Inertial
   <xacro:macro name="default_inertial" params="z_value i_value mass">
     <inertial>
@@ -21,5 +22,5 @@
                izz="${i_value}" />
     </inertial>
-  </xacro:macro>
+  </xacro:macro> -->
   <!-- Importing End-Effector -->
   <!--Arguments-->
@@ -31,5 +32,5 @@
   <xacro:include filename="$(find tiago_description)/urdf/end_effector/end_effector.urdf.xacro" />
   <xacro:include filename="$(find tiago_description_calibration)/urdf/calibration/calibration_constants.urdf.xacro" />
-  <xacro:tiago_end_effector name="${end_effector_name}" parent="top_link" type="${end_effector}" reflect="1"/>
+  <xacro:tiago_end_effector name="${end_effector_name}" parent="camera_link" type="${end_effector}" reflect="1"/>
   <!-- Include Gazebo tags -->
   <xacro:include filename="$(find arm_description)/gazebo/arm_stand_gazebo.urdf.xacro"/>
@@ -55,6 +56,14 @@
       </geometry>
     </collision>
-    <xacro:default_inertial z_value="${height1/2}"
-    i_value="1.0" mass="1"/>
+    <inertial>
+      <origin xyz="0 0 ${height1/2}" rpy="0 0 0"/>
+      <mass value="1"/>
+      <inertia
+        ixx="1.0" ixy="0.0" ixz="0.0"
+        iyy="1.0" iyz="0.0"
+        izz="1.0"/>
+    </inertial>
+    <!-- <xacro:default_inertial z_value="${height1/2}"
+    i_value="1.0" mass="1"/> -->
   </link>
   <!-- Joint between Base Link and Middle Link -->
@@ -82,6 +91,14 @@
       </geometry>
     </collision>
-    <xacro:default_inertial z_value="${height2/2 - axle_offset}"
-      i_value="1.0" mass="1"/>
+    <inertial>
+      <origin xyz="0 0 ${height2/2 - axle_offset}" rpy="0 0 0"/>
+      <mass value="1"/>
+      <inertia
+        ixx="1.0" ixy="0.0" ixz="0.0"
+        iyy="1.0" iyz="0.0"
+        izz="1.0"/>
+    </inertial>
+    <!-- <xacro:default_inertial z_value="${height2/2 - axle_offset}"
+      i_value="1.0" mass="1"/> -->
   </link>
   <!-- Joint between Middle Link and Top Link 3DOF -->
@@ -133,5 +150,5 @@
       <dynamics damping="${damp}" />
   </joint>
-  <!-- Top Link -->
+  <!-- <Top Link -->
   <link name="top_link">
     <visual>
@@ -148,6 +165,41 @@
       </geometry>
     </collision>
-    <xacro:default_inertial z_value="${height3/2 - axle_offset}"
-      i_value="1.0" mass="1"/>
+    <inertial>
+      <origin xyz="0 0 ${height3/2 - axle_offset}" rpy="0 0 0"/>
+      <mass value="1"/>
+      <inertia
+        ixx="1.0" ixy="0.0" ixz="0.0"
+        iyy="1.0" iyz="0.0"
+        izz="1.0"/>
+    </inertial>
+    <!--< xacro:default_inertial z_value="${height3/2 - axle_offset}"
+      i_value="1.0" mass="1"/> -->
+  </link>
+  <joint name="camera_joint" type="fixed">
+    <axis xyz="1 0 0" />
+    <origin xyz="${camera_link} 0 ${height3 - axle_offset*2}" rpy="0 0 0"/>
+    <parent link="top_link"/>
+    <child link="camera_link"/>
+  </joint>
+  <!-- Camera Link -->
+  <link name="camera_link">
+    <collision>
+      <origin xyz="0 0 0" rpy="0 0 0"/>
+      <geometry>
+    <box size="${camera_link} ${camera_link} ${camera_link}"/>
+      </geometry>
+    </collision>
+    <visual>
+      <origin xyz="0 0 0" rpy="0 0 0"/>
+      <geometry>
+    <box size="${camera_link} ${camera_link} ${camera_link}"/>
+      </geometry>
+      <material name="white"/>
+    </visual>
+    <inertial>
+      <mass value="1e-5" />
+      <origin xyz="0 0 0" rpy="0 0 0"/>
+      <inertia ixx="1e-6" ixy="0" ixz="0" iyy="1e-6" iyz="0" izz="1e-6" />
+    </inertial>
   </link>
  <!-- <joint name="hand_joint" type="revolute">

Commit message: Activate controllers--hand wobbles and falls--PID??

File: sim_env_ws/src/arm_description/gazebo/arm_stand_gazebo.urdf.xacro (robot description, xacro)
@@ -17,5 +17,5 @@
     <material>Gazebo/Red</material>
   </gazebo>
-  <!-- ros_control plugin
+  <!-- ros_control plugin -->
   <gazebo>
     <plugin name="gazebo_ros_control" filename="libgazebo_ros_control.so">
@@ -23,5 +23,5 @@
       <robotSimType>gazebo_ros_control/DefaultRobotHWSim</robotSimType>
     </plugin>
-  </gazebo>-->
+  </gazebo>
   <gazebo reference="camera_link">
     <sensor type="camera" name="camera1">

File: sim_env_ws/src/arm_description/urdf/arm_stand.urdf.xacro (robot description, xacro)
@@ -2,4 +2,10 @@
 <!-- Revolute-Revolute Manipulator -->
 <robot xmlns:xacro="http://www.ros.org/wiki/xacro" name="arm_stand">
+  <gazebo reference='joint_mid_top'>
+    <preserveFixedJoint>true</preserveFixedJoint>
+  </gazebo>
+  <gazebo reference='camera_joint'>
+    <preserveFixedJoint>true</preserveFixedJoint>
+  </gazebo>
   <!-- Constants for robot dimensions -->
   <xacro:property name="width" value="0.1" />
@@ -8,5 +14,6 @@
   <xacro:property name="height3" value="0.5" />
   <xacro:property name="axle_offset" value="0.05" />
-  <xacro:property name="damp" value="0.7" />
+  <xacro:property name="damp" value="0" />
+  <xacro:property name="friction" value="0.1" />
   <xacro:property name="camera_link" value="0.05" />
   <!-- Size of square 'camera' box -->
@@ -65,7 +72,17 @@
     <origin xyz="0 ${width} ${height1 - axle_offset}" rpy="0 0 0"/>
     <axis xyz="0 1 0" />
-    <dynamics damping="${damp}" />
+    <dynamics damping="${damp}" friction = "${friction}" />
     <limit effort="100.0" velocity="0.5" lower="-3.14" upper="3.14"/>
   </joint>
+  <transmission name="trans_base_mid">
+    <type>transmission_interface/SimpleTransmission</type>
+    <joint name="joint_base_mid">
+      <hardwareInterface>hardware_interface/EffortJointInterface</hardwareInterface>
+    </joint>
+    <actuator name="motor_base_mid">
+      <hardwareInterface>hardware_interface/EffortJointInterface</hardwareInterface>
+      <mechanicalReduction>1</mechanicalReduction>
+    </actuator>
+  </transmission>
   <!-- Middle Link -->
   <link name="mid_link">
@@ -92,5 +109,5 @@
     <origin xyz="0 ${width} ${height2 - axle_offset*2}" rpy="0 0 0"/>
     <!--<axis xyz="0 1 0" />
-    <dynamics damping="${damp}" />
+    <dynamics damping="${damp}" friction = "${friction}" />
     <limit effort="100.0" velocity="0.5" lower="-3.14" upper="3.14"/>-->
   </joint>
@@ -105,7 +122,18 @@
       <parent link="ball_link" />
       <child link="ball_link_psi_link" />
+      <!--<limit effort="100.0" velocity="0.5" lower="-3.14" upper="3.14"/>-->
       <axis xyz="0 0 1" />
-      <dynamics damping="${damp}" />
-  </joint>
+      <dynamics damping="${damp}" friction = "${friction}" />
+  </joint>
+  <transmission name="trans_mid_top_psi">
+    <type>transmission_interface/SimpleTransmission</type>
+    <joint name="joint_mid_top_psi">
+      <hardwareInterface>hardware_interface/EffortJointInterface</hardwareInterface>
+    </joint>
+    <actuator name="motor_mid_top_psi">
+      <hardwareInterface>hardware_interface/EffortJointInterface</hardwareInterface>
+      <mechanicalReduction>1</mechanicalReduction>
+    </actuator>
+  </transmission>
   <link name="ball_link_psi_link" >
     <inertial>
@@ -118,7 +146,18 @@
       <parent link="ball_link_psi_link"/>
       <child link="ball_link_theta_link"/>
+      <!--<limit effort="100.0" velocity="0.5" lower="-3.14" upper="3.14"/>-->
       <axis xyz="0 1 0" />
-      <dynamics damping="${damp}" />
-  </joint>
+      <dynamics damping="${damp}" friction = "${friction}" />
+  </joint>
+  <transmission name="trans_mid_top_theta">
+    <type>transmission_interface/SimpleTransmission</type>
+    <joint name="joint_mid_top_theta">
+      <hardwareInterface>hardware_interface/EffortJointInterface</hardwareInterface>
+    </joint>
+    <actuator name="motor_mid_top_theta">
+      <hardwareInterface>hardware_interface/EffortJointInterface</hardwareInterface>
+      <mechanicalReduction>1</mechanicalReduction>
+    </actuator>
+  </transmission>
   <link name="ball_link_theta_link" >
     <inertial>
@@ -128,11 +167,22 @@
     </inertial>
   </link>
-  <joint name="joint_mid_top__phi" type="continuous" >
+  <joint name="joint_mid_top_phi" type="continuous" >
       <parent link="ball_link_theta_link"/>
       <child link="top_link"/>
       <axis xyz="1 0 0" />
-      <dynamics damping="${damp}" />
-  </joint>
-  <!-- <Top Link -->
+      <!--<limit effort="100.0" velocity="0.5" lower="-3.14" upper="3.14"/>-->
+      <dynamics damping="${damp}" friction = "${friction}" />
+  </joint>
+  <transmission name="trans_mid_top_phi">
+    <type>transmission_interface/SimpleTransmission</type>
+    <joint name="joint_mid_top_phi">
+      <hardwareInterface>hardware_interface/EffortJointInterface</hardwareInterface>
+    </joint>
+    <actuator name="motor_mid_top_phi">
+      <hardwareInterface>hardware_interface/EffortJointInterface</hardwareInterface>
+      <mechanicalReduction>1</mechanicalReduction>
+    </actuator>
+  </transmission>
+  <!-- Top Link -->
   <link name="top_link">
     <visual>
@@ -156,4 +206,5 @@
     <parent link="top_link"/>
     <child link="camera_link"/>
+    <dynamics damping="${damp}" friction = "${friction}" />
   </joint>
   <!-- Camera Link -->
@@ -166,5 +217,5 @@
     </collision>
     <visual>
-      <origin xyz="0 0 ${camera_link + axle_offset/2}" rpy="0 0 0"/>
+      <origin xyz="0 0 ${camera_link + camera_link/2}" rpy="0 0 0"/>
       <geometry>
         <box size="${camera_link} ${camera_link} ${camera_link}"/>

File: sim_env_ws/src/tiago_description_complete/hey5_description/urdf/actuators.urdf.xacro (robot description, xacro)
@@ -90,5 +90,6 @@
       </actuator>
       <joint name="${name}_joint" >
-        <hardwareInterface>hardware_interface/PositionJointInterface</hardwareInterface>
+        <!--<hardwareInterface>hardware_interface/PositionJointInterface</hardwareInterface>-->
+        <hardwareInterface>hardware_interface/EffortJointInterface</hardwareInterface>
       </joint>
     </transmission>

File: sim_env_ws/src/tiago_description_complete/hey5_description/urdf/transmissions.urdf.xacro (robot description, xacro)
@@ -35,5 +35,6 @@
         <saturationLower>${jnt_abd_start}</saturationLower>
         <saturationUpper>${jnt_abd_stop}</saturationUpper>
-        <hardwareInterface>hardware_interface/JointStateInterface</hardwareInterface>
+        <!--<hardwareInterface>hardware_interface/JointStateInterface</hardwareInterface>-->
+        <hardwareInterface>hardware_interface/EffortJointInterface</hardwareInterface>
       </joint>
       <actuator name="${act_name}">
@@ -47,5 +48,6 @@
         <saturationLower>0.0</saturationLower>
         <deadBandUpper>${act_flex_start}</deadBandUpper>
-        <hardwareInterface>hardware_interface/JointStateInterface</hardwareInterface>
+        <!--<hardwareInterface>hardware_interface/JointStateInterface</hardwareInterface>-->
+        <hardwareInterface>hardware_interface/EffortJointInterface</hardwareInterface>
       </joint>
       <actuator name="${act_name}">
@@ -58,5 +60,6 @@
         <saturationLower>0.0</saturationLower>
         <deadBandUpper>${act_flex_start}</deadBandUpper>
-        <hardwareInterface>hardware_interface/JointStateInterface</hardwareInterface>
+        <!--<hardwareInterface>hardware_interface/JointStateInterface</hardwareInterface>-->
+        <hardwareInterface>hardware_interface/EffortJointInterface</hardwareInterface>
       </joint>
       <actuator name="${act_name}">
@@ -70,5 +73,6 @@
         <saturationLower>0.0</saturationLower>
         <deadBandUpper>${act_flex_start}</deadBandUpper>
-        <hardwareInterface>hardware_interface/JointStateInterface</hardwareInterface>
+        <!--<hardwareInterface>hardware_interface/JointStateInterface</hardwareInterface>-->
+        <hardwareInterface>hardware_interface/EffortJointInterface</hardwareInterface>
       </joint>
       <actuator name="${act_name}">
@@ -81,5 +85,6 @@
         <saturationLower>0.0</saturationLower>
         <deadBandUpper>${act_flex_start}</deadBandUpper>
-        <hardwareInterface>hardware_interface/JointStateInterface</hardwareInterface>
+        <!--<hardwareInterface>hardware_interface/JointStateInterface</hardwareInterface>-->
+        <hardwareInterface>hardware_interface/EffortJointInterface</hardwareInterface>
       </joint>
       <actuator name="${act_name}">
@@ -113,5 +118,6 @@
         <saturationLower>${jnt_abd_start}</saturationLower>
         <saturationUpper>${jnt_abd_stop}</saturationUpper>
-        <hardwareInterface>hardware_interface/JointStateInterface</hardwareInterface>
+        <!--<hardwareInterface>hardware_interface/JointStateInterface</hardwareInterface>-->
+        <hardwareInterface>hardware_interface/EffortJointInterface</hardwareInterface>
       </joint>
       <actuator name="${act_name}">
@@ -125,5 +131,6 @@
         <saturationLower>0.0</saturationLower>
         <deadBandUpper>${act_flex_start}</deadBandUpper>
-        <hardwareInterface>hardware_interface/JointStateInterface</hardwareInterface>
+        <!--<hardwareInterface>hardware_interface/JointStateInterface</hardwareInterface>-->
+        <hardwareInterface>hardware_interface/EffortJointInterface</hardwareInterface>
       </joint>
       <actuator name="${act_name}">
@@ -136,5 +143,6 @@
         <saturationLower>0.0</saturationLower>
         <deadBandUpper>${act_flex_start}</deadBandUpper>
-        <hardwareInterface>hardware_interface/JointStateInterface</hardwareInterface>
+        <!--<hardwareInterface>hardware_interface/JointStateInterface</hardwareInterface>-->
+        <hardwareInterface>hardware_interface/EffortJointInterface</hardwareInterface>
       </joint>
       <actuator name="${act_name}">
@@ -148,5 +156,6 @@
         <saturationLower>0.0</saturationLower>
         <deadBandUpper>${act_flex_start}</deadBandUpper>
-        <hardwareInterface>hardware_interface/JointStateInterface</hardwareInterface>
+        <!--<hardwareInterface>hardware_interface/JointStateInterface</hardwareInterface>-->
+        <hardwareInterface>hardware_interface/EffortJointInterface</hardwareInterface>
       </joint>
       <actuator name="${act_name}">
@@ -159,5 +168,6 @@
         <saturationLower>0.0</saturationLower>
         <deadBandUpper>${act_flex_start}</deadBandUpper>
-        <hardwareInterface>hardware_interface/JointStateInterface</hardwareInterface>
+        <!--<hardwareInterface>hardware_interface/JointStateInterface</hardwareInterface>-->
+        <hardwareInterface>hardware_interface/EffortJointInterface</hardwareInterface>
       </joint>
       <actuator name="${act_name}">
@@ -171,5 +181,6 @@
         <saturationLower>0.0</saturationLower>
         <deadBandUpper>${act_flex_start}</deadBandUpper>
-        <hardwareInterface>hardware_interface/JointStateInterface</hardwareInterface>
+        <!--<hardwareInterface>hardware_interface/JointStateInterface</hardwareInterface>-->
+        <hardwareInterface>hardware_interface/EffortJointInterface</hardwareInterface>
       </joint>
       <actuator name="${act_name}">
@@ -182,5 +193,6 @@
         <saturationLower>0.0</saturationLower>
         <deadBandUpper>${act_flex_start}</deadBandUpper>
-        <hardwareInterface>hardware_interface/JointStateInterface</hardwareInterface>
+        <!--<hardwareInterface>hardware_interface/JointStateInterface</hardwareInterface>-->
+        <hardwareInterface>hardware_interface/EffortJointInterface</hardwareInterface>
       </joint>
       <actuator name="${act_name}">
