Commit message: re-built arm so it doesnt rotate in air---still falls under gravity

File: sim_env_ws/src/arm_description/gazebo/arm_stand_gazebo.urdf.xacro (robot description, xacro)
@@ -3,4 +3,5 @@
   <!-- Base Link -->
   <gazebo reference="base_link">
+    <!--<gravity>false</gravity>-->
     <material>Gazebo/White</material>
   </gazebo>
@@ -10,4 +11,6 @@
     <mu2>0.2</mu2>
     <material>Gazebo/Green</material>
+    <!--<turnGravityOff>true</turnGravityOff>-->
+    <gravity>false</gravity>
   </gazebo>
   <!-- Top Link -->
@@ -16,5 +19,22 @@
     <mu2>0.2</mu2>
     <material>Gazebo/Red</material>
+    <gravity>false</gravity>
   </gazebo>
+  <!-- Fore Link -->
+  <gazebo reference="fore_link">
+    <mu1>0.2</mu1>
+    <mu2>0.2</mu2>
+    <material>Gazebo/Blue</material>
+    <!--<gravity>false</gravity>-->
+  </gazebo>
+  <!--<gazebo reference="hand_palm_link">
+    <gravity>false</gravity>
+  </gazebo>
+  <gazebo reference="hand_tool_link">
+    <gravity>false</gravity>
+  </gazebo>
+  <gazebo reference="hand_safety_box">
+    <gravity>false</gravity>
+  </gazebo>-->
   <!-- ros_control plugin -->
   <gazebo>
@@ -25,4 +45,5 @@
   </gazebo>
   <gazebo reference="camera_link">
+    <gravity>false</gravity>
     <sensor type="camera" name="camera1">
       <update_rate>30.0</update_rate>
@@ -40,7 +61,7 @@
         <noise>
           <type>gaussian</type>
-          <!-- Noise is sampled independently per pixel on each frame.
+          <!--Noise is sampled independently per pixel on each frame.
                That pixel's noise value is added to each of its color
-               channels, which at that point lie in the range [0,1]. -->
+               channels, which at that point lie in the range [0,1].-->
           <mean>0.0</mean>
           <stddev>0.007</stddev>

File: sim_env_ws/src/arm_description/urdf/arm_stand.urdf (robot description, URDF)
Before this commit: robot arm_stand, 48 links, 47 joints
Links:
- removed link ball_link
- removed link ball_link_psi_link
- removed link ball_link_theta_link
- added link fore_link, mass 1; collision box size=0.5 0.1 0.1; visual box size=0.5 0.1 0.1
- link top_link: geometry collision box size=0.5 0.1 0.1; visual box size=0.5 0.1 0.1
Joints:
- removed joint joint_mid_top__phi
- removed joint joint_mid_top_psi
- removed joint joint_mid_top_theta
- added joint joint_top_fore: type revolute, parent top_link, child fore_link, origin xyz=0.45 0 0 rpy=0 0 0, axis 1 0 0, limit lower=-3.14 upper=3.14 effort=1000.0 velocity=0.5
- joint camera_joint: origin xyz=0 0 0.4 rpy=0 1.57 -1.57 -> xyz=0.45 0 0 rpy=0 0 0; parent top_link -> fore_link
- joint hand_palm_joint: origin xyz=0 0 0.45 rpy=0 -1.57 0 -> xyz=0.5 0 0 rpy=-1.57 0 0; parent top_link -> fore_link
- joint hand_safety_box_joint: origin xyz=0 0 0.45 rpy=0 -1.57 0 -> xyz=0.5 0 0 rpy=-1.57 0 0; parent top_link -> fore_link
- joint hand_tool_joint: origin xyz=0 0 0.45 rpy=0 -1.57 0 -> xyz=0.5 0 0 rpy=-1.57 0 0; parent top_link -> fore_link
- joint joint_base_mid: limit lower=-3.14 upper=3.14 effort=100.0 velocity=0.5 -> lower=-3.14 upper=3.14 effort=1000.0 velocity=0.5
- joint joint_mid_top: axis (none) -> 0 0 1; child ball_link -> top_link; limit (none) -> lower=-3.14 upper=3.14 effort=1000.0 velocity=0.5; origin xyz=0 0.1 0.4 rpy=0 0 0 -> xyz=0 0 0.5 rpy=0 0 0; type fixed -> revolute

File: sim_env_ws/src/arm_description/urdf/old_arm_stand.urdf.xacro (robot description, xacro)
@@ -2,4 +2,10 @@
 <!-- Revolute-Revolute Manipulator -->
 <robot xmlns:xacro="http://www.ros.org/wiki/xacro" name="arm_stand">
+  <gazebo reference='joint_mid_top'>
+    <preserveFixedJoint>true</preserveFixedJoint>
+  </gazebo>
+  <gazebo reference='camera_joint'>
+    <preserveFixedJoint>true</preserveFixedJoint>
+  </gazebo>
   <!-- Constants for robot dimensions -->
   <xacro:property name="PI" value="3.1415926535897931"/>
@@ -10,8 +16,11 @@
   <xacro:property name="height3" value="0.5" />
   <xacro:property name="axle_offset" value="0.05" />
-  <xacro:property name="damp" value="0.7" />
-  <xacro:property name="friction" value="0" />
+  <xacro:property name="damp" value="10" />
+  <xacro:property name="friction" value="0.1" />
   <xacro:property name="camera_link" value="0.05" />
   <!-- Size of square 'camera' box -->
+  <!-- Import Rviz colors -->
+  <xacro:include
+      filename="$(find arm_description)/urdf/materials.urdf.xacro" />
   <!-- Default Inertial -->
   <xacro:macro name="default_inertial" params="z_value height mass width">
@@ -24,9 +33,4 @@
     </inertial>
   </xacro:macro>
-  <!-- Import Rviz colors -->
-  <xacro:include
-      filename="$(find arm_description)/urdf/materials.urdf.xacro" />
-  <!-- Include Gazebo tags -->
-  <xacro:include filename="$(find arm_description)/gazebo/arm_stand_gazebo.urdf.xacro"/>
   <!-- Importing End-Effector -->
   <!--Arguments-->
@@ -38,5 +42,7 @@
   <xacro:include filename="$(find tiago_description)/urdf/end_effector/end_effector.urdf.xacro" />
   <xacro:include filename="$(find tiago_description_calibration)/urdf/calibration/calibration_constants.urdf.xacro" />
-  <xacro:tiago_end_effector name="${end_effector_name}" parent="fore_link" type="${end_effector}" reflect="1"/>
+  <xacro:tiago_end_effector name="${end_effector_name}" parent="top_link" type="${end_effector}" reflect="1"/>
+  <!-- Include Gazebo tags -->
+  <xacro:include filename="$(find arm_description)/gazebo/arm_stand_gazebo.urdf.xacro"/>
   <!--Arm Stand-->
   <link name="world"/>
@@ -71,4 +77,14 @@
     <limit effort="1000.0" velocity="0.5" lower="-3.14" upper="3.14"/>
   </joint>
+  <transmission name="trans_base_mid">
+    <type>transmission_interface/SimpleTransmission</type>
+    <joint name="joint_base_mid">
+      <hardwareInterface>hardware_interface/EffortJointInterface</hardwareInterface>
+    </joint>
+    <actuator name="motor_base_mid">
+      <hardwareInterface>hardware_interface/EffortJointInterface</hardwareInterface>
+      <mechanicalReduction>1</mechanicalReduction>
+    </actuator>
+  </transmission>
   <!-- Middle Link -->
   <link name="mid_link">
@@ -89,74 +105,110 @@
     height="${height2}" mass="${mass}" width = "${width}"/>
   </link>
-  <!-- Joint between Middle Link and Top Link -->
-  <joint name="joint_mid_top" type="revolute">
+  <!-- Joint between Middle Link and Top Link 3DOF -->
+  <joint name="joint_mid_top" type="fixed">
     <parent link="mid_link" />
-    <child link="top_link" />
-    <origin xyz="0 0 ${height2}" rpy="0 0 0"/>
-    <axis xyz="0 0 1" />
+    <child link="ball_link" />
+    <origin xyz="0 ${width} ${height2 - axle_offset*2}" rpy="0 0 0"/>
+    <!--<axis xyz="0 1 0" />
     <dynamics damping="${damp}" friction = "${friction}" />
-    <limit effort="1000.0" velocity="0.5" lower="-3.14" upper="3.14"/>
-  </joint>
+    <limit effort="100.0" velocity="0.5" lower="-3.14" upper="3.14"/>-->
+  </joint>
+  <link name="ball_link">
+    <inertial>
+      <mass value="1e-5" />
+      <origin xyz="0 0 0" rpy="0 0 0"/>
+      <inertia ixx="1e-6" ixy="0" ixz="0" iyy="1e-6" iyz="0" izz="1e-6" />
+    </inertial>
+  </link>
+  <joint name="joint_mid_top_psi" type="continuous" >
+      <parent link="ball_link" />
+      <child link="ball_link_psi_link" />
+      <!--<limit effort="100.0" velocity="0.5" lower="-3.14" upper="3.14"/>-->
+      <axis xyz="0 0 1" />
+      <dynamics damping="${damp}" friction = "${friction}" />
+  </joint>
+  <transmission name="trans_mid_top_psi">
+    <type>transmission_interface/SimpleTransmission</type>
+    <joint name="joint_mid_top_psi">
+      <hardwareInterface>hardware_interface/EffortJointInterface</hardwareInterface>
+    </joint>
+    <actuator name="motor_mid_top_psi">
+      <hardwareInterface>hardware_interface/EffortJointInterface</hardwareInterface>
+      <mechanicalReduction>1</mechanicalReduction>
+    </actuator>
+  </transmission>
+  <link name="ball_link_psi_link" >
+    <inertial>
+      <mass value="1e-5" />
+      <origin xyz="0 0 0" rpy="0 0 0"/>
+      <inertia ixx="1e-6" ixy="0" ixz="0" iyy="1e-6" iyz="0" izz="1e-6" />
+    </inertial>
+  </link>
+  <joint name="joint_mid_top_theta" type="continuous" >
+      <parent link="ball_link_psi_link"/>
+      <child link="ball_link_theta_link"/>
+      <!--<limit effort="100.0" velocity="0.5" lower="-3.14" upper="3.14"/>-->
+      <axis xyz="0 1 0" />
+      <dynamics damping="${damp}" friction = "${friction}" />
+  </joint>
+  <transmission name="trans_mid_top_theta">
+    <type>transmission_interface/SimpleTransmission</type>
+    <joint name="joint_mid_top_theta">
+      <hardwareInterface>hardware_interface/EffortJointInterface</hardwareInterface>
+    </joint>
+    <actuator name="motor_mid_top_theta">
+      <hardwareInterface>hardware_interface/EffortJointInterface</hardwareInterface>
+      <mechanicalReduction>1</mechanicalReduction>
+    </actuator>
+  </transmission>
+  <link name="ball_link_theta_link" >
+    <inertial>
+      <mass value="1e-5" />
+      <origin xyz="0 0 0" rpy="0 0 0"/>
+      <inertia ixx="1e-6" ixy="0" ixz="0" iyy="1e-6" iyz="0" izz="1e-6" />
+    </inertial>
+  </link>
+  <joint name="joint_mid_top_phi" type="continuous" >
+      <parent link="ball_link_theta_link"/>
+      <child link="top_link"/>
+      <axis xyz="1 0 0" />
+      <!--<limit effort="100.0" velocity="0.5" lower="-3.14" upper="3.14"/>-->
+      <dynamics damping="${damp}" friction = "${friction}" />
+  </joint>
+  <transmission name="trans_mid_top_phi">
+    <type>transmission_interface/SimpleTransmission</type>
+    <joint name="joint_mid_top_phi">
+      <hardwareInterface>hardware_interface/EffortJointInterface</hardwareInterface>
+    </joint>
+    <actuator name="motor_mid_top_phi">
+      <hardwareInterface>hardware_interface/EffortJointInterface</hardwareInterface>
+      <mechanicalReduction>1</mechanicalReduction>
+    </actuator>
+  </transmission>
   <!-- Top Link -->
   <link name="top_link">
     <visual>
-      <origin xyz="${height3/2 - axle_offset} 0 0" rpy="0 0 0" />
-      <geometry>
-        <box size="${height3} ${width} ${width}" />
+      <origin xyz="0 0 ${height3/2 - axle_offset}" rpy="0 0 0" />
+      <geometry>
+        <box size="${width} ${width} ${height3}" />
       </geometry>
       <material name="red"/>
     </visual>
     <collision>
-      <origin xyz="${height3/2 - axle_offset} 0 0" rpy="0 0 0" />
-      <geometry>
-        <box size="${height3} ${width} ${width}" />
-      </geometry>
-    </collision>
-    <inertial>
-      <origin xyz="${height3/2 - axle_offset} 0 0" rpy="0 0 0"/>
-      <mass value="${mass}"/>
-      <inertia ixx="${0.0833333 * mass * (0 + 0)}" ixy="0.0" ixz="0.0"
-        iyy="${0.0833333 * mass * (height3)*(height3)}" iyz="0.0"
-        izz="${0.0833333 * mass * (height3)*(height3)}" />
-    </inertial>
-  </link>
-  <!-- Joint between Top Link and Forearm Link -->
-  <joint name="joint_top_fore" type="revolute">
-    <parent link="top_link" />
-    <child link="fore_link" />
-    <origin xyz="${height3 - axle_offset} 0 0" rpy="0 0 0"/>
-    <axis xyz="1 0 0" />
-    <dynamics damping="${damp}" friction = "${friction}" />
-    <limit effort="1000.0" velocity="0.5" lower="-3.14" upper="3.14"/>
-  </joint>
-  <link name="fore_link">
-    <visual>
-      <origin xyz="${height3/2} 0 0" rpy="0 0 0" />
-      <geometry>
-        <box size="${height3} ${width} ${width}" />
-      </geometry>
-      <material name="blue"/>
-    </visual>
-    <collision>
-      <origin xyz="${height3/2} 0 0" rpy="0 0 0" />
-      <geometry>
-        <box size="${height3} ${width} ${width}" />
-      </geometry>
-    </collision>
-    <inertial>
-      <origin xyz="${height3/2} 0 0" rpy="0 0 0"/>
-      <mass value="${mass}"/>
-      <inertia ixx="${0.0833333 * mass * (0 + 0)}" ixy="0.0" ixz="0.0"
-        iyy="${0.0833333 * mass * (height3)*(height3)}" iyz="0.0"
-        izz="${0.0833333 * mass * (height3)*(height3)}" />
-    </inertial>
+      <origin xyz="0 0 ${height3/2 - axle_offset}" rpy="0 0 0" />
+      <geometry>
+        <box size="${width} ${width} ${height3}" />
+      </geometry>
+    </collision>
+    <xacro:default_inertial z_value="${height3/2 - axle_offset}"
+      height="${height3}" mass="${mass}" width = "${width}"/>
   </link>
   <joint name="camera_joint" type="fixed">
-    <origin xyz="${height3 - axle_offset} 0 0" rpy="0 0 0"/>
-    <parent link="fore_link"/>
+    <origin xyz="0 0 ${height2 - axle_offset*2}" rpy="0 1.57 -1.57"/>
+    <parent link="top_link"/>
     <child link="camera_link"/>
     <dynamics damping="${damp}" friction = "${friction}" />
   </joint>
-   <!--Camera Link-->
+  <!-- Camera Link -->
   <link name="camera_link">
     <collision>
@@ -179,44 +231,4 @@
     </inertial>
   </link>
-  <!--Transmission-->
-  <transmission name="trans_base_mid">
-    <type>transmission_interface/SimpleTransmission</type>
-    <joint name="joint_base_mid">
-      <hardwareInterface>hardware_interface/EffortJointInterface</hardwareInterface>
-    </joint>
-    <actuator name="motor_base_mid">
-      <hardwareInterface>hardware_interface/EffortJointInterface</hardwareInterface>
-      <mechanicalReduction>1</mechanicalReduction>
-    </actuator>
-  </transmission>
-  <transmission name="trans_mid_top">
-    <type>transmission_interface/SimpleTransmission</type>
-    <joint name="joint_mid_top">
-      <hardwareInterface>hardware_interface/EffortJointInterface</hardwareInterface>
-    </joint>
-    <actuator name="motor_mid_top">
-      <hardwareInterface>hardware_interface/EffortJointInterface</hardwareInterface>
-      <mechanicalReduction>1</mechanicalReduction>
-    </actuator>
-  </transmission>
-  <transmission name="trans_top_fore">
-    <type>transmission_interface/SimpleTransmission</type>
-    <joint name="joint_top_fore">
-      <hardwareInterface>hardware_interface/EffortJointInterface</hardwareInterface>
-    </joint>
-    <actuator name="motor_top_fore">
-      <hardwareInterface>hardware_interface/EffortJointInterface</hardwareInterface>
-      <mechanicalReduction>1</mechanicalReduction>
-    </actuator>
-  </transmission>
-  <xacro:macro name="box_inertial_with_origin" params="x y z mass *origin">
-    <inertial>
-      <mass value="${mass}" />
-      <insert_block name="origin" />
-      <inertia ixx="${0.0833333 * mass * (y*y + z*z)}" ixy="0.0" ixz="0.0"
-        iyy="${0.0833333 * mass * (x*x + z*z)}" iyz="0.0"
-        izz="${0.0833333 * mass * (x*x + y*y)}" />
-    </inertial>
-  </xacro:macro>
  <!-- <joint name="hand_joint" type="revolute">
     <parent link="top_link"/>

File: sim_env_ws/src/tiago_description_complete/tiago_robot/tiago_description/urdf/end_effector/end_effector.urdf.xacro (robot description, xacro)
@@ -44,5 +44,5 @@
   <xacro:if value="${type == 'pal-hey5'}">
     <xacro:hey5_hand parent="${parent}" name="${name}" reflect="${reflect}">
-      <origin xyz="0 0 ${height2 - axle_offset}" rpy="0 -1.57 0"/>
+      <origin xyz="${height3} 0 0" rpy="-1.57 0 0"/>
       <!--<origin xyz="0 0 0" rpy="0 0 0"/>-->
     </xacro:hey5_hand>
@@ -50,5 +50,5 @@
       <parent link="${parent}"/>
       <child link="${name}_safety_box"/>
-      <origin xyz="0 0 ${height2 - axle_offset}" rpy="0 -1.57 0"/>
+      <origin xyz="${height3} 0 0" rpy="-1.57 0 0"/>
       <!--<origin xyz="0.1 0.02 ${reflect * 0.02}" rpy="0 0 0"/>-->
     </joint>

Commit message: moveIt in RVIZ control thru python, commandline, rviz GUI --need gazebo connection

File: sim_env_ws/src/arm_description/gazebo/arm_stand_gazebo.urdf.xacro (robot description, xacro)
@@ -1,4 +1,6 @@
 <?xml version="1.0"?>
-<robot xmlns:xacro="http://ros.org/wiki/xacro">
+<robot xmlns:xacro="http://ros.org/wiki/xacro"
+       xmlns:controller="http://playerstage.sourceforge.net/gazebo/xmlschema/#controller"
+       xmlns:interface="http://playerstage.sourceforge.net/gazebo/xmlschema/#interface">
   <gazebo reference='camera_joint'>
     <preserveFixedJoint>true</preserveFixedJoint>

File: sim_env_ws/src/tiago_description_complete/hey5_description/urdf/fingers.urdf.xacro (robot description, xacro)
@@ -127,5 +127,6 @@
         <origin xyz="0 0 0" rpy="0 0 0" />
         <geometry>
-          <mesh filename="package://hey5_description/meshes/finger_abd_collision.stl" scale="1 1 ${reflect}" />
+        <!--////////////////////////////////////////////////////////////////////////////////////////////////////////////11-->
+          <mesh filename="package://hey5_description/meshes/finger_abd_collision.stl" scale="0.01 0.01 ${reflect}" />
         </geometry>
       </collision>
@@ -168,5 +169,6 @@
         <origin xyz="0 0 0" rpy="0 0 0" />
         <geometry>
-          <mesh filename="package://hey5_description/meshes/thumb_abd_collision.stl" scale="1 ${reflect} 1" />
+        <!--/////////////////////////////////////////////////////////////////////////////////////////////////////////////11-->
+          <mesh filename="package://hey5_description/meshes/thumb_abd_collision.stl" scale="0.01 ${reflect} 0.01" />
         </geometry>
       </collision>
@@ -253,5 +255,6 @@
         <origin xyz="0 0 0" rpy="0 0 0" />
         <geometry>
-          <mesh filename="package://hey5_description/meshes/finger_flex_collision.stl" />
+        <!--//////////////////////////////////////////////////////////////////////////////////////////////nothing-->
+          <mesh filename="package://hey5_description/meshes/finger_flex_collision.stl" scale = "0.01 0.01 0.01"/>
         </geometry>
       </collision>
@@ -296,5 +299,6 @@
         <origin xyz="0 0 0" rpy="0 0 0" />
         <geometry>
-          <mesh filename="package://hey5_description/meshes/finger_flex_tip_collision.stl" />
+        <!--///////////////////////////////////////////////////////////////////////////////////////NOTHING-->
+          <mesh filename="package://hey5_description/meshes/finger_flex_tip_collision.stl" scale="0.01 0.01 0.01"/>
         </geometry>
       </collision>

File: sim_env_ws/src/tiago_description_complete/hey5_description/urdf/palm.urdf.xacro (robot description, xacro)
@@ -40,5 +40,6 @@
         <origin xyz="0 0 0" rpy="0 0 0" />
         <geometry>
-          <mesh filename="package://hey5_description/meshes/palm_collision.stl" scale="1 1 ${reflect}" />
+        <!--///////////////////////////////////////////////////////////////////////////////////////////////////////11-->
+          <mesh filename="package://hey5_description/meshes/palm_collision.stl" scale="0.1 0.1 ${reflect}" />
         </geometry>
       </collision>

File: sim_env_ws/src/tiago_description_complete/tiago_robot/tiago_description/urdf/end_effector/end_effector.urdf.xacro (robot description, xacro)
@@ -70,5 +70,5 @@
         <origin xyz="0 0 0" rpy="0 0 0" />
         <geometry>
-          <box size="0.2 0.115 0.18" />
+          <box size="0.02 0.0115 0.018" />
         </geometry>
       </collision>
